Commit message: should be ok

File: urdf/d435.gazebo.xacro (robot description, xacro)
@@ -112,5 +112,5 @@
     </gazebo>
     <gazebo>
-      <plugin name="${topics_ns}" filename="librealsense_gazebo_plugin.so">
+      <plugin name="${topics_ns}" filename="libd435_gazebo.so">
         <prefix>${camera_name}</prefix>
       	<depthUpdateRate>60.0</depthUpdateRate>

File: urdf/d435.urdf.xacro (robot description, xacro)
@@ -8,5 +8,5 @@
 <robot name="sensor_d435" xmlns:xacro="http://ros.org/wiki/xacro">
   <!--File includes-->
-  <xacro:include filename="$(find realsense_gazebo_plugin)/urdf/d435.gazebo.xacro"/>
+  <xacro:include filename="$(find d435_gazebo)/urdf/d435.gazebo.xacro"/>
   <xacro:macro name="sensor_d435" params="name:=camera topics_ns:=camera parent *origin">
     <xacro:property name="M_PI" value="3.1415926535897931" />
@@ -48,5 +48,5 @@
         <geometry>
           <!-- <box size="${d435_cam_width} ${d435_cam_height} ${d435_cam_depth}"/> -->
-          <mesh filename="package://realsense_gazebo_plugin/models/realsense_camera/meshes/realsense.dae" />
+          <mesh filename="package://d435_gazebo/models/realsense_camera/meshes/realsense.dae" />
           <!--<mesh filename="package://realsense2_description/meshes/d435/d435.dae" />-->
         </geometry>

File: urdf/d435_simulation.xacro (robot description, xacro)
@@ -7,5 +7,5 @@
     <link name="world"/>
     <!-- Import macro for realsense-RS200 camera-->
-    <xacro:include filename="$(find realsense_gazebo_plugin)/urdf/d435.urdf.xacro"/>
+    <xacro:include filename="$(find d435_gazebo)/urdf/d435.urdf.xacro"/>
     <!-- Create camera instance -->
     <xacro:sensor_d435 parent="world">
